Commit message: feat:多机械臂，IK方法

File: arm_description/urdf/lbr_iiwa_14_r820.xacro (robot description, xacro)
@@ -1,7 +1,9 @@
 <?xml version="1.0"?>
 <robot name="kuka_lbr_iiwa_14_r820" xmlns:xacro="http://wiki.ros.org/xacro">
+  <xacro:arg name="origin_xyz" default="0 0 0"/>
+  <xacro:arg name="origin_rpy" default="0 0 0"/>
   <!-- ✅ 引入宏定义 -->
   <xacro:include filename="$(find arm_description)/urdf/lbr_iiwa_14_r820_macro.xacro"/>
   <!-- ✅ 调用宏，传入前缀 -->
-  <xacro:kuka_lbr_iiwa_14_r820 prefix="lbr_iiwa_"/>
+  <xacro:kuka_lbr_iiwa_14_r820 prefix="lbr_iiwa_" origin_xyz="$(arg origin_xyz)" origin_rpy="$(arg origin_rpy)"/>
 </robot>

File: arm_description/urdf/lbr_iiwa_14_r820_macro.xacro (robot description, xacro)
@@ -1,5 +1,5 @@
 <?xml version="1.0"?>
 <robot xmlns:xacro="http://wiki.ros.org/xacro">
-  <xacro:macro name="kuka_lbr_iiwa_14_r820" params="prefix">
+  <xacro:macro name="kuka_lbr_iiwa_14_r820" params="prefix origin_xyz:='0 0 0' origin_rpy:='0 0 0'">
   <link name="world"/>
     <!-- link list -->
@@ -221,7 +221,34 @@
   <limit lower="-3.0541" upper="3.0541" effort="200" velocity="2.356" />
 </joint>
-<!-- ✅ 新增末端滑动关节（沿世界 X 方向） -->
-  <!-- Gazebo 扩展：让轴方向固定在世界坐标 -->
-<!-- ✅ 固定连接到世界 -->
+  <!-- Payload (2kg) -->
+  <joint name="${prefix}payload_joint" type="fixed">
+    <parent link="${prefix}link_7"/>
+    <child link="${prefix}payload_link"/>
+    <origin xyz="0 0 0.2" rpy="0 0 0"/>
+  </joint>
+  <link name="${prefix}payload_link">
+    <inertial>
+      <origin xyz="0 0 0" rpy="0 0 0"/>
+      <mass value="2.0"/>
+      <inertia ixx="0.01" ixy="0" ixz="0" iyy="0.01" iyz="0" izz="0.01"/>
+    </inertial>
+    <visual>
+      <origin xyz="0 0 0" rpy="0 0 0"/>
+      <geometry>
+        <box size="0.1 0.1 0.1"/>
+      </geometry>
+      <material name="payload_grey">
+        <color rgba="0.5 0.5 0.5 1.0"/>
+      </material>
+    </visual>
+    <collision>
+      <geometry>
+        <box size="0.1 0.1 0.1"/>
+      </geometry>
+    </collision>
+  </link>
+  <gazebo reference="${prefix}payload_link">
+    <material>Gazebo/Grey</material>
+  </gazebo>
 <link name="${prefix}base" />
 <joint name="${prefix}base_link-base" type="fixed">
@@ -233,5 +260,5 @@
   <parent link="world"/>
   <child link="${prefix}base_link"/>
-  <origin xyz="0 0 0" rpy="0 0 0"/>
+  <origin xyz="${origin_xyz}" rpy="${origin_rpy}"/>
 </joint>
       <!-- ================== transmissions ================== -->
@@ -303,5 +330,5 @@
 <gazebo>
   <plugin name="gazebo_ros_control" filename="libgazebo_ros_control.so">
-    <robotNamespace>/</robotNamespace>
+    <!-- <robotNamespace>/</robotNamespace> REMOVED to allow namespacing -->
     <robotSimType>gazebo_ros_control/DefaultRobotHWSim</robotSimType>
     <gravity_compensation>false</gravity_compensation>
